File: wearable_cape.sch (KiCad schematic (older format))
At the start: 66 parts, among them J1 J1 0 5, J2 J2 2 3, J3 J3 1 4, P1 BELA_AINS, P2 SERIAL_BREAKOUT, P3 CONN_01X02_BATTERY, P4 BELA_AOUTS, P5 PWR_OUT_AMPS, P6 STATUS_BREAKOUT, P7 A_IN_BREAKOUT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

Commit message: updates - wiring mistake!
Parts:
- added JP1: serial power select, jcr-device:SolderJumper-3_P1.3mm_Open_Pad1.0x1.5mm, symbol wearable_cape-rescue:SolderJumper_3_Open-jcr-device
- added JP2: analog power select, jcr-device:SolderJumper-3_P1.3mm_Open_Pad1.0x1.5mm, symbol wearable_cape-rescue:SolderJumper_3_Open-jcr-device
- C1, C10, C11, C14, C15, C16, C17, C2, C20, C3, C4, C5, C8, C9: symbol Device:C -> wearable_cape-rescue:C-Device
- C12, C13, C18, C19, C21, C22, C6, C7: symbol Device:CP1 -> wearable_cape-rescue:CP1-Device
- C23, C24, C25: symbol jcr-device:C_Ceramic -> wearable_cape-rescue:C_Ceramic-jcr-device
- C26: symbol jcr-device:C -> wearable_cape-rescue:C-jcr-device
- P3: symbol jcr-conn:CONN_01X02_BATTERY -> wearable_cape-rescue:CONN_01X02_BATTERY-jcr-conn
- P6, P7: symbol wearable_cape:CONN_02X04_UNI -> wearable_cape:CONN_01x08_UNI
- R1, R10, R11, R12, R13, R14, R15, R16, R35, R36, R37, R38, R39, R4, R40, R5, R6, R7, R8, R9: symbol Device:R -> wearable_cape-rescue:R-Device
- U5: symbol jcr-ic:MAX6100 -> wearable_cape-rescue:MAX6100-jcr-ic
Connections:
- net BELA_IN0: now also P7.3 (Pin_3); no longer P7.8 (P8)
- net BELA_IN1: now also P7.4 (Pin_4); no longer P7.7 (P7)
- net BELA_IN2: now also P7.5 (Pin_5); no longer P7.6 (P6)
- net BELA_IN3: now also P7.6 (Pin_6); no longer P7.5 (P5)
- net BELA_IN4: now also P7.7 (Pin_7); no longer P7.4 (P4)
- net BELA_IN5: now also P7.8 (Pin_8); no longer P7.3 (P3)
- net D0: now also P6.4 (Pin_4); no longer P6.8 (P8)
- net D11: now also P6.5 (Pin_5); no longer P6.3 (P3)
- net D8: now also P6.6 (Pin_6); no longer P6.5 (P5)
- net STATUS_LED: now also P6.8 (Pin_8); no longer P6.2 (P2)
- net SYS_3.3V: now also P6.3 (Pin_3), JP1.1 (A), JP2.3 (B); no longer P6.6 (P6)
- net SYS_5V: now also JP1.3 (B), JP2.1 (A); no longer P2.1 (P1), P7.2 (P2)
- net ~SW_HALT: now also P6.2 (Pin_2); no longer P6.4 (P4)
- new net: JP1.2 (C), P2.1 (P1)
- new net: JP2.2 (C), P7.2 (Pin_2)
Other:
- note added: "NOTE: Bela Digital Pins are 3.3V tolerant!!\nYou must level shift the serial signal coming\nback to the Bela down to 3.3V!"
- note added: "NOTE: SYS3v3 is much quieter than 5V\nadd a LDO regulator on daughter boards for clean\npower from 5V"
- note added: "NOTE: SYS_5V supply on the BeagleBone Black is the regulated \nsupply coming from the USB port. It will always be available \nregardless of how the BeagleBone is powered, but it has a limit \nof 250mA of current."
- note added: "NOTE: VDD_5V supply on the BeagleBone Black is only available \nwhen powered from the DC barrel connector (or other external \nsource). Given a suitable power supply, these pins can supply \nup to 1A of current. These are the pins used to power the audio \namplifiers on the Bela cape."
- note removed: "NOTE: add a LDO regulator\non daughter boards for clean\npower"
- note removed: "blue"
- note removed: "green"
- note removed: "red"
- moved on the sheet: P9

Commit message: updates to v2 schematics with notations on wiring errors
Parts:
- added D?: RGB_LED, symbol JCR_DEVICE:RGB_LED
- added D?: 2mA GRN LED, symbol JCR_DEVICE:LED
- added P?: CONN_02X04_UNI, symbol wearable_cape:CONN_02X04_UNI
- added R?: 47, symbol JCR_DEVICE:R_Small
- P6: value STATUS_BREAKOUT -> WRONG:STATUS_BREAKOUT
Connections:
- net GND: now also P?.7 (P7), R?.2
- net STATUS_LED: now also D?.2 (A), P?.8 (P8)
- new net: D?.2 (COM), R?.1
- new net 3v3: D?.1 (K)
- new net BLUE_LED: D?.4 (BLU), P?.5 (P5)
- new net GREEN_LED: D?.3 (GRN), P?.3 (P3)
- new net MODE_SEL1_3v3: P?.2 (P2)
- new net MODE_SEL2: P?.4 (P4)
- new net RED_LED: D?.1 (RED), P?.1 (P1)
- new net SW_HALT: P?.6 (P6)
Other:
- note added: "How can these labels possibly be correct? D0 and SYS5v?"
- note added: "NEW BREAKOUTBOARD CONNECTOR & BREAKOUT"
- note added: "These buttons are incorrectly labeled on the v2 boards"
- note added: "WARNING: This is not how the status breakout \nis wired on the actual V2 boards!"
- note added: "\nThe actual wiring of the status header on the v2 board is...\n\n1 GND\n2 STATUS_LED\n3 D11\n4 SW_HALT\n5 D8\n6 MODE_SEL1 / 3v3\n7 D9\n8 MODE_SEL2"
- moved on the sheet: C25, C26, JP2, P6, P7, P8, P9, R1, R12, SW1, SW2, U2C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
